File: actuation.sch (KiCad schematic (older format))
At the start: 0 parts

Commit message: Changes: 1. Relay and partial analog sensing circuitry added.
Parts:
- added J?: Fan, symbol Connector:Conn_01x02_Male
- added K? (x2): Songle-SRD, Relay_THT:Relay_SPDT_SANYOU_SRD_Series_Form_C, symbol Custom_Misc:Songle-SRD
- added U?: ULN2803A, symbol Transistor_Array:ULN2803A
Connections:
- net labels added: Fan_Ctrl, Gnd, RL1_C, RL1_NC, RL1_NO, RL2_C, RL2_NC, RL2_NO, Relay1_Ctrl, Relay2_Ctrl, V_Coil
- wire segments 0 -> 43
Changed lines of the file:
@@
 $Descr A4 11693 8268
 encoding utf-8
-Sheet 1 7
+Sheet 4 7
 Title ""
 Date "2018-09-29"
@@
 Comment4 ""
 $EndDescr
+$Comp
+L Transistor_Array:ULN2803A U?
+U 1 1 5BB0992C
+P 4500 2650
+F 0 "U?" H 4500 3217 50  0000 C CNN
+F 1 "ULN2803A" H 4500 3126 50  0000 C CNN
+F 2 "" H 4550 2000 50  0001 L CNN
+F 3 "http://www.ti.com/lit/ds/symlink/uln2803a.pdf" H 4600 2450 50  0001 C CNN
+	1    4500 2650
+	1    0    0    -1
+$EndComp
+Text HLabel 5000 1350 1    50   Input ~ 0
+V_Coil
+Wire Wire Line
+	5000 1350 5000 1450
+Wire Wire Line
+	5000 2350 4900 2350
+Wire Wire Line
+	5350 1550 5350 1450
+Wire Wire Line
+	5350 1450 5000 1450
+Connection ~ 5000 1450
+Wire Wire Line
+	5000 1450 5000 2350
+Wire Wire Line
+	4900 2450 5350 2450
+Wire Wire Line
+	5350 2450 5350 2150
+Wire Wire Line
+	4900 2550 5350 2550
+Wire Wire Line
+	5350 2550 5350 2450
+Connection ~ 5350 2450
+Wire Wire Line
+	4900 2650 5350 2650
+Wire Wire Line
+	5350 2650 5350 2550
+Connection ~ 5350 2550
+Wire Wire Line
+	4900 3150 5350 3150
+Wire Wire Line
+	5350 3150 5350 3400
+Wire Wire Line
+	4900 3050 5350 3050
+Wire Wire Line
+	5350 3050 5350 3150
+Connection ~ 5350 3150
+Wire Wire Line
+	4900 2950 5350 2950
+Wire Wire Line
+	5350 2950 5350 3050
+Connection ~ 5350 3050
+Text HLabel 5050 4350 3    50   Input ~ 0
+V_Coil
+Wire Wire Line
+	5050 4350 5050 4200
+Wire Wire Line
+	5050 4200 5350 4200
+Wire Wire Line
+	5350 4200 5350 4000
+$Comp
+L Connector:Conn_01x02_Male J?
+U 1 1 5BB0A132
+P 6700 2750
+F 0 "J?" H 6672 2723 50  0000 R CNN
+F 1 "Fan" H 6672 2632 50  0000 R CNN
+F 2 "" H 6700 2750 50  0001 C CNN
+F 3 "~" H 6700 2750 50  0001 C CNN
+	1    6700 2750
+	-1   0    0    -1
+$EndComp
+Wire Wire Line
+	4900 2850 5350 2850
+Wire Wire Line
+	4900 2750 5350 2750
+Wire Wire Line
+	5350 2750 5350 2850
+Connection ~ 5350 2850
+Wire Wire Line
+	5350 2850 6500 2850
+Text HLabel 6250 2750 0    50   Input ~ 0
+V_Coil
+Wire Wire Line
+	6250 2750 6500 2750
+Text HLabel 4300 3500 0    50   BiDi ~ 0
+Gnd
+Wire Wire Line
+	4300 3500 4500 3500
+Wire Wire Line
+	4500 3500 4500 3350
+Text HLabel 3800 2450 0    50   Input ~ 0
+Relay1_Ctrl
+Text HLabel 3800 2850 0    50   Input ~ 0
+Fan_Ctrl
+Text HLabel 3800 3150 0    50   Input ~ 0
+Relay2_Ctrl
+Wire Wire Line
+	3800 2450 3900 2450
+Wire Wire Line
+	4100 2550 3900 2550
+Wire Wire Line
+	3900 2550 3900 2450
+Connection ~ 3900 2450
+Wire Wire Line
+	3900 2450 4100 2450
+Wire Wire Line
+	4100 2650 3900 2650
+Wire Wire Line
+	3900 2650 3900 2550
+Connection ~ 3900 2550
+Wire Wire Line
+	3800 2850 3900 2850
+Wire Wire Line
+	4100 2750 3900 2750
+Wire Wire Line
+	3900 2750 3900 2850
+Connection ~ 3900 2850
+Wire Wire Line
+	3900 2850 4100 2850
+Wire Wire Line
+	4100 3150 3900 3150
+Wire Wire Line
+	4100 3050 3900 3050
+Wire Wire Line
+	3900 3050 3900 3150
+Connection ~ 3900 3150
+Wire Wire Line
+	3900 3150 3800 3150
+Wire Wire Line
+	4100 2950 3900 2950
+Wire Wire Line
+	3900 2950 3900 3050
+Connection ~ 3900 3050
+$Comp
+L Custom_Misc:Songle-SRD K?
+U 1 1 5BB11D63
+P 5500 1850
+F 0 "K?" H 5980 1896 50  0000 L CNN
+F 1 "Songle-SRD" H 5980 1805 50  0000 L CNN
+F 2 "Relay_THT:Relay_SPDT_SANYOU_SRD_Series_Form_C" H 5550 1450 50  0001 C CNN
+F 3 "https://www.mycomkits.com/reference/Songle_SRD(T73)_Relay.pdf" H 5550 1450 50  0001 C CNN
+	1    5500 1850
+	1    0    0    -1
+$EndComp
+$Comp
+L Custom_Misc:Songle-SRD K?
+U 1 1 5BB11DAF
+P 5500 3700
+F 0 "K?" H 5980 3746 50  0000 L CNN
+F 1 "Songle-SRD" H 5980 3655 50  0000 L CNN
+F 2 "Relay_THT:Relay_SPDT_SANYOU_SRD_Series_Form_C" H 5550 3300 50  0001 C CNN
+F 3 "https://www.mycomkits.com/reference/Songle_SRD(T73)_Relay.pdf" H 5550 3300 50  0001 C CNN
+	1    5500 3700
+	1    0    0    -1
+$EndComp
+Text HLabel 5850 1550 1    50   BiDi ~ 0
+RL1_NO
+Text HLabel 5650 1550 1    50   BiDi ~ 0
+RL1_NC
+Text HLabel 5750 2150 3    50   BiDi ~ 0
+RL1_C
+Text HLabel 5750 4000 3    50   BiDi ~ 0
+RL2_C
+Text HLabel 5650 3400 1    50   BiDi ~ 0
+RL2_NC
+Text HLabel 5850 3400 1    50   BiDi ~ 0
+RL2_NO
 $EndSCHEMATC

Commit message: Changes: 1. Added all component footprints
Parts:
- J14: renamed from J?; footprint (none) -> Connector_JST:JST_EH_B02B-EH-A_1x02_P2.50mm_Vertical
- U4: renamed from U?; footprint (none) -> Package_SO:SOIC-18W_7.5x11.6mm_P1.27mm
- gave numbers to parts that had none: 2
Changed lines of the file:
@@
 $EndDescr
 $Comp
-L Transistor_Array:ULN2803A U?
+L Transistor_Array:ULN2803A U4
 U 1 1 5BB0992C
 P 4500 2650
-F 0 "U?" H 4500 3217 50  0000 C CNN
+F 0 "U4" H 4500 3217 50  0000 C CNN
 F 1 "ULN2803A" H 4500 3126 50  0000 C CNN
-F 2 "" H 4550 2000 50  0001 L CNN
+F 2 "Package_SO:SOIC-18W_7.5x11.6mm_P1.27mm" H 4550 2000 50  0001 L CNN
 F 3 "http://www.ti.com/lit/ds/symlink/uln2803a.pdf" H 4600 2450 50  0001 C CNN
 	1    4500 2650
@@
 	5350 4200 5350 4000
 $Comp
-L Connector:Conn_01x02_Male J?
+L Connector:Conn_01x02_Male J14
 U 1 1 5BB0A132
 P 6700 2750
-F 0 "J?" H 6672 2723 50  0000 R CNN
+F 0 "J14" H 6672 2723 50  0000 R CNN
 F 1 "Fan" H 6672 2632 50  0000 R CNN
-F 2 "" H 6700 2750 50  0001 C CNN
+F 2 "Connector_JST:JST_EH_B02B-EH-A_1x02_P2.50mm_Vertical" H 6700 2750 50  0001 C CNN
 F 3 "~" H 6700 2750 50  0001 C CNN
 	1    6700 2750
@@
 Connection ~ 3900 3050
 $Comp
-L Custom_Misc:Songle-SRD K?
+L Custom_Misc:Songle-SRD K1
 U 1 1 5BB11D63
 P 5500 1850
-F 0 "K?" H 5980 1896 50  0000 L CNN
+F 0 "K1" H 5980 1896 50  0000 L CNN
 F 1 "Songle-SRD" H 5980 1805 50  0000 L CNN
 F 2 "Relay_THT:Relay_SPDT_SANYOU_SRD_Series_Form_C" H 5550 1450 50  0001 C CNN
@@
 $EndComp
 $Comp
-L Custom_Misc:Songle-SRD K?
+L Custom_Misc:Songle-SRD K2
 U 1 1 5BB11DAF
 P 5500 3700
-F 0 "K?" H 5980 3746 50  0000 L CNN
+F 0 "K2" H 5980 3746 50  0000 L CNN
 F 1 "Songle-SRD" H 5980 3655 50  0000 L CNN
 F 2 "Relay_THT:Relay_SPDT_SANYOU_SRD_Series_Form_C" H 5550 3300 50  0001 C CNN
