File: serial.sch (KiCad schematic (older format))
At the start: 0 parts

Commit message: Changes: 1. Serial (RS232, 485) circuit added.
Parts:
- added C?: 0.1uF, symbol Device:C
- added C? (x2): 1nF, symbol Device:C_Small
- added C? (x5): 0.1uF, symbol Device:CP1_Small
- added D?: MMBD914, Package_TO_SOT_SMD:SOT-23, symbol Diode:BAV99
- added D? (x3): TVS, symbol Device:D_TVS_ALT
- added D_RX, D_TX: LED, symbol Device:LED_Small
- added F? (x2): PPTC, symbol Device:Polyfuse_Small
- added R?: 1K, symbol Device:R
- added R? (x2): 1K, symbol Device:R_Small
- added R?: 120, symbol Device:R_Small
- added R_RX, R_TX: 330, symbol Device:R_Small
- added SW?: SW_DIP_x04, symbol Switch:SW_DIP_x04
- added U?: MAX232, symbol Interface_UART:MAX232
- added U?: 74HC14, symbol 74xx:74HC14
- added U?: SN65LBC176D, Package_SO:SOIC-8_3.9x4.9mm_P1.27mm, symbol Interface_UART:SN65LBC176D
Connections:
- net labels added: GND, RS232_RX, RS232_TX, RS485_A+, RS485_B-, UART_RX, UART_TX, VCC
- wire segments 0 -> 109
- no-connect marks 0 -> 4

Commit message: Changes: 1. Digital sensing circuit added.
Changed lines of the file:
@@
 Title ""
 Date "2018-09-29"
-Rev "0.2"
+Rev "0.3"
 Comp "Bodhileaf Technologies"
 Comment1 ""
@@
 Wire Wire Line
 	5200 5050 5550 5050
-Text HLabel 4500 5750 0    50   Input ~ 0
+Text HLabel 4500 5750 0    50   BiDi ~ 0
 GND
 Text HLabel 4700 650  0    50   Input ~ 0
@@
 Text HLabel 1650 3700 0    50   Input ~ 0
 UART_TX
-Text HLabel 1650 3900 0    50   Input ~ 0
+Text HLabel 1650 3900 0    50   Output ~ 0
 UART_RX
-Text HLabel 8950 4400 2    50   Input ~ 0
+Text HLabel 8950 4400 2    50   BiDi ~ 0
 RS485_A+
-Text HLabel 8950 3900 2    50   Input ~ 0
+Text HLabel 8950 3900 2    50   BiDi ~ 0
 RS485_B-
 Wire Wire Line
@@
 Wire Wire Line
 	4900 5750 4900 5550
-Text HLabel 6550 4900 0    50   Input ~ 0
+Text HLabel 6550 4900 0    50   BiDi ~ 0
 GND
 Wire Wire Line
@@
 Wire Wire Line
 	6250 4100 6250 3800
-Text HLabel 6600 2250 2    50   Input ~ 0
+Text HLabel 6600 2250 2    50   Output ~ 0
 RS232_TX
 Text HLabel 6600 2650 2    50   Input ~ 0
@@
 Wire Wire Line
 	8450 4400 8600 4400
-Text HLabel 5000 3500 0    50   Input ~ 0
+Text HLabel 5000 3500 0    50   BiDi ~ 0
 GND
 Wire Wire Line
@@
 Wire Wire Line
 	5900 1900 6000 1900
-Text HLabel 6600 2100 2    50   Input ~ 0
+Text HLabel 6600 2100 2    50   BiDi ~ 0
 GND
 Wire Wire Line
@@
 	5900 650  5900 750
 Connection ~ 5100 650
-Text HLabel 6200 1100 2    50   Input ~ 0
+Text HLabel 6200 1100 2    50   BiDi ~ 0
 GND
 Wire Wire Line

Commit message: Changes: 1. Added all component footprints
Parts:
- removed C? (x5): 0.1uF, symbol Device:CP1_Small
- added C3, C5, C6, C7, C8: 0.1uF, Capacitor_SMD:C_1206_3216Metric, symbol Device:C_Small
- C10, C9: renamed from C?; footprint (none) -> Capacitor_SMD:C_0805_2012Metric
- C4: renamed from C?; footprint (none) -> Capacitor_SMD:C_1206_3216Metric
- D3: renamed from D?; footprint Package_TO_SOT_SMD:SOT-23 -> Diode_SMD:D_SOT-23_ANK
- D4, D5, D6: renamed from D?; footprint (none) -> Diode_SMD:D_SMB
- D_RX1: renamed from D_RX; footprint (none) -> LED_SMD:LED_0805_2012Metric
- D_TX1: renamed from D_TX; footprint (none) -> LED_SMD:LED_0805_2012Metric
- F2, F3: renamed from F?; footprint (none) -> Fuse:Fuse_1812_4532Metric
- R16, R17, R18, R19: renamed from R?; footprint (none) -> Resistor_SMD:R_0805_2012Metric
- R_RX1: renamed from R_RX; footprint (none) -> Resistor_SMD:R_0805_2012Metric
- R_TX1: renamed from R_TX; footprint (none) -> Resistor_SMD:R_0805_2012Metric
- SW2: renamed from SW?; footprint (none) -> Button_Switch_SMD:SW_DIP_SPSTx04_Slide_KingTek_DSHP04TJ_W5.25mm_P1.27mm_JPin
- U1: renamed from U?; footprint (none) -> Package_SO:TSSOP-14_4.4x5mm_P0.65mm
- U7: renamed from U?; footprint (none) -> Package_SO:TSSOP-16_4.4x5mm_P0.65mm
- gave numbers to parts that had none: 1

Commit message: Changes: 1. Removed TVS diodes in favour of a RS485 transceiver of the same footprint that contains ESD protection 2. Tried different layouts.
Parts:
- removed D3: MMBD914, Diode_SMD:D_SOT-23_ANK, symbol Diode:BAV99
- removed D4, D5, D6: TVS, Diode_SMD:D_SMB, symbol Device:D_TVS_ALT
- added D3: MMBD914, Diode_SMD:D_SOT-23_ANK, symbol Diode:1N914WT
- C3, C4, C5, C6, C7, C8: footprint Capacitor_SMD:C_1206_3216Metric -> Capacitor_SMD:C_0805_2012Metric
- U8: value SN65LBC176D -> SN65HVD75DR
Connections:
- wire segments 109 -> 99
Changed lines of the file:
@@
 P 6700 4000
 F 0 "U8" H 6800 3650 50  0000 C CNN
-F 1 "SN65LBC176D" H 7000 4350 50  0000 C CNN
+F 1 "SN65HVD75DR" H 7000 4350 50  0000 C CNN
 F 2 "Package_SO:SOIC-8_3.9x4.9mm_P1.27mm" H 6700 3500 50  0001 C CNN
 F 3 "http://www.ti.com/lit/ds/symlink/sn75lbc176.pdf" H 8300 3800 50  0001 C CNN
 	1    6700 4000
 	1    0    0    -1
-$EndComp
-$Comp
-L Diode:BAV99 D3
-U 1 1 5BAEE1D7
-P 5200 4750
-F 0 "D3" V 5154 4828 50  0000 L CNN
-F 1 "MMBD914" V 5245 4828 50  0000 L CNN
-F 2 "Diode_SMD:D_SOT-23_ANK" H 5200 4600 50  0001 C CNN
-F 3 "www.nxp.com/documents/data_sheet/BAV99_SER.pdf" H 5200 4850 50  0001 C CNN
-	1    5200 4750
-	0    1    1    0
 $EndComp
 $Comp
@@
 F 0 "C4" H 5015 5446 50  0000 L CNN
 F 1 "0.1uF" H 5015 5355 50  0000 L CNN
-F 2 "Capacitor_SMD:C_1206_3216Metric" H 4938 5250 50  0001 C CNN
+F 2 "Capacitor_SMD:C_0805_2012Metric" H 4938 5250 50  0001 C CNN
 F 3 "~" H 4900 5400 50  0001 C CNN
 	1    4900 5400
@@
 	1    0    0    -1
 $EndComp
-$Comp
-L Device:D_TVS_ALT D4
-U 1 1 5BAF4329
-P 8150 3650
-F 0 "D4" V 8104 3729 50  0000 L CNN
-F 1 "TVS" V 8195 3729 50  0000 L CNN
-F 2 "Diode_SMD:D_SMB" H 8150 3650 50  0001 C CNN
-F 3 "~" H 8150 3650 50  0001 C CNN
-	1    8150 3650
-	0    1    1    0
-$EndComp
-$Comp
-L Device:D_TVS_ALT D5
-U 1 1 5BAF452A
-P 8150 4150
-F 0 "D5" V 8104 4229 50  0000 L CNN
-F 1 "TVS" V 8195 4229 50  0000 L CNN
-F 2 "Diode_SMD:D_SMB" H 8150 4150 50  0001 C CNN
-F 3 "~" H 8150 4150 50  0001 C CNN
-	1    8150 4150
-	0    1    1    0
-$EndComp
-$Comp
-L Device:D_TVS_ALT D6
-U 1 1 5BAF456C
-P 8150 4650
-F 0 "D6" V 8104 4729 50  0000 L CNN
-F 1 "TVS" V 8195 4729 50  0000 L CNN
-F 2 "Diode_SMD:D_SMB" H 8150 4650 50  0001 C CNN
-F 3 "~" H 8150 4650 50  0001 C CNN
-	1    8150 4650
-	0    1    1    0
-$EndComp
 Wire Wire Line
 	7000 4100 7350 4100
@@
 	7950 4100 7950 3900
 Wire Wire Line
-	7950 3900 8150 3900
-Wire Wire Line
 	7000 4200 7350 4200
 Wire Wire Line
 	7950 4200 7950 4400
-Wire Wire Line
-	7950 4400 8150 4400
-Wire Wire Line
-	8150 4000 8150 3900
-Connection ~ 8150 3900
 Wire Wire Line
 	7350 4050 7350 4100
@@
 	7650 4900 7350 4900
 Connection ~ 7350 4900
-Wire Wire Line
-	8150 4300 8150 4400
-Connection ~ 8150 4400
-Wire Wire Line
-	8150 3800 8150 3900
-Wire Wire Line
-	8150 4500 8150 4400
-Wire Wire Line
-	8150 4800 8150 4900
-Wire Wire Line
-	8150 4900 7650 4900
-Connection ~ 7650 4900
-Wire Wire Line
-	7650 3400 8150 3400
-Wire Wire Line
-	8150 3400 8150 3500
-Connection ~ 7650 3400
 Wire Wire Line
 	6700 4400 6700 4900
@@
 $EndComp
 Wire Wire Line
-	8150 3900 8450 3900
-Wire Wire Line
 	8800 3900 8950 3900
 Wire Wire Line
 	8800 4400 8950 4400
-Wire Wire Line
-	8150 4400 8450 4400
 Wire Wire Line
 	8450 4050 8450 3900
@@
 F 0 "C5" H 5992 896 50  0000 L CNN
 F 1 "0.1uF" H 5992 805 50  0000 L CNN
-F 2 "Capacitor_SMD:C_1206_3216Metric" H 5900 850 50  0001 C CNN
+F 2 "Capacitor_SMD:C_0805_2012Metric" H 5900 850 50  0001 C CNN
 F 3 "~" H 5900 850 50  0001 C CNN
 	1    5900 850
@@
 F 0 "C7" H 6292 1446 50  0000 L CNN
 F 1 "0.1uF" H 6292 1355 50  0000 L CNN
-F 2 "Capacitor_SMD:C_1206_3216Metric" H 6200 1400 50  0001 C CNN
+F 2 "Capacitor_SMD:C_0805_2012Metric" H 6200 1400 50  0001 C CNN
 F 3 "~" H 6200 1400 50  0001 C CNN
 	1    6200 1400
@@
 F 0 "C6" H 6092 2046 50  0000 L CNN
 F 1 "0.1uF" H 6092 1955 50  0000 L CNN
-F 2 "Capacitor_SMD:C_1206_3216Metric" H 6000 2000 50  0001 C CNN
+F 2 "Capacitor_SMD:C_0805_2012Metric" H 6000 2000 50  0001 C CNN
 F 3 "~" H 6000 2000 50  0001 C CNN
 	1    6000 2000
@@
 F 0 "C8" H 6442 1896 50  0000 L CNN
 F 1 "0.1uF" H 6442 1805 50  0000 L CNN
-F 2 "Capacitor_SMD:C_1206_3216Metric" H 6350 1850 50  0001 C CNN
+F 2 "Capacitor_SMD:C_0805_2012Metric" H 6350 1850 50  0001 C CNN
 F 3 "~" H 6350 1850 50  0001 C CNN
 	1    6350 1850
@@
 F 0 "C3" H 4142 1446 50  0000 L CNN
 F 1 "0.1uF" H 4142 1355 50  0000 L CNN
-F 2 "Capacitor_SMD:C_1206_3216Metric" H 4050 1400 50  0001 C CNN
+F 2 "Capacitor_SMD:C_0805_2012Metric" H 4050 1400 50  0001 C CNN
 F 3 "~" H 4050 1400 50  0001 C CNN
 	1    4050 1400
 	1    0    0    -1
 $EndComp
+Wire Wire Line
+	7950 3900 8450 3900
+Wire Wire Line
+	7950 4400 8450 4400
+$Comp
+L Diode:1N914WT D3
+U 1 1 5BB68902
+P 5200 4750
+F 0 "D3" V 5154 4830 50  0000 L CNN
+F 1 "MMBD914" V 5245 4830 50  0000 L CNN
+F 2 "Diode_SMD:D_SOT-23_ANK" H 5200 4575 50  0001 C CNN
+F 3 "http://www.mouser.com/ds/2/149/1N4148WT-461550.pdf" H 5200 4750 50  0001 C CNN
+	1    5200 4750
+	0    1    1    0
+$EndComp
 $EndSCHEMATC

Commit message: Changes: 1. Some net names, connector names changed to be more meaningful 2. I2C connector added 3. Mistake in power bank bypass connection rectified 4. Layout changed. Almost finalized.
Connections:
- net labels added: DGND
- wire segments 99 -> 100
Changed lines of the file:
@@
 Sheet 7 7
 Title ""
-Date "2018-10-02"
-Rev "0.6"
+Date "2018-10-05"
+Rev "0.7"
 Comp "Bodhileaf Technologies"
 Comment1 ""
@@
 	0    1    1    0
 $EndComp
+Text HLabel 7900 4900 2    50   Output ~ 0
+DGND
+Wire Wire Line
+	7650 4900 7900 4900
+Connection ~ 7650 4900
 $EndSCHEMATC
