File: serial.sch (KiCad schematic (older format))
At the start: 23 parts, among them SW2 SW_DIP_x04, U1 74HC14, U7 MAX232, U8 SN65HVD75DR

Commit message: Changes: 1. Added a power LED 2. Added PPTC to the inputs of optocoupler 3. Added PPTC to the transceiver side of the RS232 driver 4. Corrected ADC footprint
Parts:
- added F4, F5: PPTC_500mA, Fuse:Fuse_1812_4532Metric, symbol Device:Polyfuse_Small
- F2, F3: value PPTC -> PPTC_500mA
Connections:
- net RS232_RX: now also F5.1; no longer U7.13 (R1IN)
- net RS232_TX: now also F4.1; no longer U7.14 (T1OUT)
- new net: F5.2, U7.13 (R1IN)
- new net: F4.2, U7.14 (T1OUT)
Changed lines of the file:
@@
 P 8700 3900
 F 0 "F2" V 8495 3900 50  0000 C CNN
-F 1 "PPTC" V 8586 3900 50  0000 C CNN
+F 1 "PPTC_500mA" V 8586 3900 50  0000 C CNN
 F 2 "Fuse:Fuse_1812_4532Metric" H 8750 3700 50  0001 L CNN
 F 3 "~" H 8700 3900 50  0001 C CNN
@@
 P 8700 4400
 F 0 "F3" V 8800 4400 50  0000 C CNN
-F 1 "PPTC" V 8900 4400 50  0000 C CNN
+F 1 "PPTC_500mA" V 8900 4400 50  0000 C CNN
 F 2 "Fuse:Fuse_1812_4532Metric" H 8750 4200 50  0001 L CNN
 F 3 "~" H 8700 4400 50  0001 C CNN
@@
 Connection ~ 1800 2950
 Wire Wire Line
-	6600 2250 5900 2250
-Wire Wire Line
-	6600 2650 5900 2650
+	6600 2250 6350 2250
+Wire Wire Line
+	6600 2650 6350 2650
 $Comp
 L Device:C_Small C5
@@
 	7650 4900 7900 4900
 Connection ~ 7650 4900
+$Comp
+L Device:Polyfuse_Small F4
+U 1 1 5BC03D49
+P 6250 2250
+F 0 "F4" V 6200 2350 50  0000 C CNN
+F 1 "PPTC_500mA" V 6350 2150 50  0000 C CNN
+F 2 "Fuse:Fuse_1812_4532Metric" H 6300 2050 50  0001 L CNN
+F 3 "~" H 6250 2250 50  0001 C CNN
+	1    6250 2250
+	0    1    1    0
+$EndComp
+Wire Wire Line
+	6150 2250 5900 2250
+$Comp
+L Device:Polyfuse_Small F5
+U 1 1 5BC040AD
+P 6250 2650
+F 0 "F5" V 6200 2750 50  0000 C CNN
+F 1 "PPTC_500mA" V 6350 2550 50  0000 C CNN
+F 2 "Fuse:Fuse_1812_4532Metric" H 6300 2450 50  0001 L CNN
+F 3 "~" H 6250 2650 50  0001 C CNN
+	1    6250 2650
+	0    1    1    0
+$EndComp
+Wire Wire Line
+	6150 2650 5900 2650
 $EndSCHEMATC

Commit message: Changes: 1. Corrected RS485 circuit connections 2. Added silk screen labels and labels to schematics
Connections:
- net at SW2.5, U8.1 (R): no longer D3.1 (K), R16.1
- net at SW2.6, U8.4 (D): now also D3.1 (K), R16.1
Changed lines of the file:
@@
 Sheet 7 7
 Title ""
-Date "2018-10-17"
-Rev "0.9"
+Date "2018-11-24"
+Rev "0.91"
 Comp "Bodhileaf Technologies"
 Comment1 ""
@@
 Text HLabel 8950 3900 2    50   BiDi ~ 0
 RS485_B-
-Wire Wire Line
-	3650 4200 4900 4200
 $Comp
 L Switch:SW_DIP_x04 SW2
@@
 	2300 3800 2450 3800
 Wire Wire Line
-	3050 3900 6400 3900
+	3050 3900 4900 3900
 Wire Wire Line
 	3050 4000 3650 4000
@@
 NoConn ~ 5900 2850
 NoConn ~ 5900 2450
-Wire Wire Line
-	5200 4600 5200 4200
-Connection ~ 5200 4200
-Wire Wire Line
-	5200 4200 6400 4200
-Wire Wire Line
-	4900 4600 4900 4200
-Connection ~ 4900 4200
-Wire Wire Line
-	4900 4200 5200 4200
 Wire Wire Line
 	4500 5750 4900 5750
@@
 Wire Wire Line
 	6150 2650 5900 2650
+Wire Wire Line
+	3650 4200 6400 4200
+Wire Wire Line
+	4900 4600 4900 3900
+Connection ~ 4900 3900
+Wire Wire Line
+	4900 3900 5200 3900
+Wire Wire Line
+	5200 4600 5200 3900
+Connection ~ 5200 3900
+Wire Wire Line
+	5200 3900 6400 3900
 $EndSCHEMATC

Commit message: Added some more labels to schematics
Parts:
- U7: value MAX232 -> SP3232EBEY
Changed lines of the file:
@@
 P 5100 2150
 F 0 "U7" H 5300 3300 50  0000 C CNN
-F 1 "MAX232" H 5300 3200 50  0000 C CNN
+F 1 "SP3232EBEY" H 5400 3200 50  0000 C CNN
 F 2 "Package_SO:TSSOP-16_4.4x5mm_P0.65mm" H 5150 1100 50  0001 L CNN
 F 3 "http://www.ti.com/lit/ds/symlink/max232.pdf" H 5100 2250 50  0001 C CNN
