File: analogSensing.sch (KiCad schematic (older format))
At the start: 0 parts

Commit message: Changes: 1. Relay and partial analog sensing circuitry added.
Parts:
- added C?: 0.1uF, 0.1uF, symbol Device:CP1_Small
- added C?: 10uF, symbol Device:CP_Small
- added U?: MCP3428, symbol Analog_ADC:MCP3428
Connections:
- net labels added: Gnd, SCL, SDA, Vcc
- wire segments 0 -> 19
Changed lines of the file:
@@
 $Descr A4 11693 8268
 encoding utf-8
-Sheet 1 7
+Sheet 5 7
 Title ""
 Date "2018-09-29"
@@
 Comment4 ""
 $EndDescr
+$Comp
+L Analog_ADC:MCP3428 U?
+U 1 1 5BB12D76
+P 4800 2900
+F 0 "U?" H 4550 3350 50  0000 C CNN
+F 1 "MCP3428" H 5050 3350 50  0000 C CNN
+F 2 "" H 4800 2900 50  0001 C CNN
+F 3 "http://ww1.microchip.com/downloads/en/DeviceDoc/22226a.pdf" H 4800 2900 50  0001 C CNN
+	1    4800 2900
+	1    0    0    -1
+$EndComp
+$Comp
+L Device:CP1_Small C?
+U 1 1 5BB12E03
+P 5500 1950
+F 0 "C?" H 5591 1996 50  0000 L CNN
+F 1 "0.1uF" H 5591 1905 50  0000 L CNN
+F 2 "0.1uF" H 5500 1950 50  0001 C CNN
+F 3 "~" H 5500 1950 50  0001 C CNN
+	1    5500 1950
+	1    0    0    -1
+$EndComp
+$Comp
+L Device:CP_Small C?
+U 1 1 5BB12EC2
+P 5100 1950
+F 0 "C?" H 5188 1996 50  0000 L CNN
+F 1 "10uF" H 5188 1905 50  0000 L CNN
+F 2 "" H 5100 1950 50  0001 C CNN
+F 3 "~" H 5100 1950 50  0001 C CNN
+	1    5100 1950
+	1    0    0    -1
+$EndComp
+Text HLabel 4800 1650 1    50   Input ~ 0
+Vcc
+Wire Wire Line
+	4800 1650 4800 1750
+Wire Wire Line
+	4800 1750 5100 1750
+Wire Wire Line
+	5100 1750 5100 1850
+Connection ~ 4800 1750
+Wire Wire Line
+	4800 1750 4800 2400
+Wire Wire Line
+	5100 1750 5500 1750
+Wire Wire Line
+	5500 1750 5500 1850
+Connection ~ 5100 1750
+Text HLabel 5350 2250 3    50   Input ~ 0
+Gnd
+Wire Wire Line
+	5100 2050 5100 2200
+Wire Wire Line
+	5100 2200 5350 2200
+Wire Wire Line
+	5350 2200 5350 2250
+Wire Wire Line
+	5350 2200 5500 2200
+Wire Wire Line
+	5500 2200 5500 2050
+Connection ~ 5350 2200
+Text HLabel 5350 3050 2    50   BiDi ~ 0
+Gnd
+Wire Wire Line
+	5200 3000 5300 3000
+Wire Wire Line
+	5300 3000 5300 3050
+Wire Wire Line
+	5300 3050 5350 3050
+Wire Wire Line
+	5200 3100 5300 3100
+Wire Wire Line
+	5300 3100 5300 3050
+Connection ~ 5300 3050
+Text HLabel 4800 3650 3    50   BiDi ~ 0
+Gnd
+Wire Wire Line
+	4800 3650 4800 3500
+Text HLabel 5350 2700 2    50   BiDi ~ 0
+SCL
+Text HLabel 5350 2800 2    50   BiDi ~ 0
+SDA
+Wire Wire Line
+	5200 2700 5350 2700
+Wire Wire Line
+	5200 2800 5350 2800
 $EndSCHEMATC

Commit message: Changes: 1. Added Analog circuitry
Parts:
- added R? (x3): 10K, symbol Device:R_Small
- added R?: 20m, symbol Device:R_Small
- added R?: 1K, symbol Device:R_Small
- added R_4_20: 100, symbol Device:R_Small
- added SW?: SW_SPDT, symbol Switch:SW_SPDT
Connections:
- net labels added: 420+, 420-, I_Sense+, I_Sense-, R_Sense, T_Sense, V_Sense
- wire segments 19 -> 59
Changed lines of the file:
@@
 Sheet 5 7
 Title ""
-Date "2018-09-29"
-Rev "0.3"
+Date "2018-10-01"
+Rev "0.4"
 Comp "Bodhileaf Technologies"
 Comment1 ""
@@
 Wire Wire Line
 	5200 2800 5350 2800
+Text HLabel 4400 2700 0    50   BiDi ~ 0
+Gnd
+Text HLabel 4400 3100 0    50   BiDi ~ 0
+Gnd
+$Comp
+L Device:R_Small R?
+U 1 1 5BB20FA7
+P 2200 2450
+F 0 "R?" H 2259 2496 50  0000 L CNN
+F 1 "10K" H 2259 2405 50  0000 L CNN
+F 2 "" H 2200 2450 50  0001 C CNN
+F 3 "~" H 2200 2450 50  0001 C CNN
+	1    2200 2450
+	1    0    0    -1
+$EndComp
+$Comp
+L Device:R_Small R?
+U 1 1 5BB20FD7
+P 2200 2750
+F 0 "R?" H 2259 2796 50  0000 L CNN
+F 1 "10K" H 2259 2705 50  0000 L CNN
+F 2 "" H 2200 2750 50  0001 C CNN
+F 3 "~" H 2200 2750 50  0001 C CNN
+	1    2200 2750
+	1    0    0    -1
+$EndComp
+Text HLabel 2200 3250 3    50   BiDi ~ 0
+Gnd
+Text HLabel 2000 2250 0    50   Input ~ 0
+V_Sense
+Wire Wire Line
+	2000 2250 2200 2250
+Wire Wire Line
+	2200 2250 2200 2350
+Wire Wire Line
+	2200 2900 2200 2850
+Wire Wire Line
+	2200 2650 2200 2600
+Connection ~ 2200 2600
+Wire Wire Line
+	2200 2600 2200 2550
+$Comp
+L Device:R_Small R?
+U 1 1 5BB21FC0
+P 2200 3000
+F 0 "R?" H 2259 3046 50  0000 L CNN
+F 1 "10K" H 2259 2955 50  0000 L CNN
+F 2 "" H 2200 3000 50  0001 C CNN
+F 3 "~" H 2200 3000 50  0001 C CNN
+	1    2200 3000
+	1    0    0    -1
+$EndComp
+Wire Wire Line
+	2200 3100 2200 3250
+$Comp
+L Device:R_Small R?
+U 1 1 5BB22A1E
+P 2800 3000
+F 0 "R?" H 2859 3046 50  0000 L CNN
+F 1 "20m" H 2859 2955 50  0000 L CNN
+F 2 "" H 2800 3000 50  0001 C CNN
+F 3 "~" H 2800 3000 50  0001 C CNN
+	1    2800 3000
+	1    0    0    -1
+$EndComp
+Wire Wire Line
+	2800 2900 2800 2800
+Text HLabel 2050 3600 0    50   Input ~ 0
+I_Sense+
+Text HLabel 2050 3750 0    50   Input ~ 0
+I_Sense-
+Wire Wire Line
+	2600 3600 2600 2800
+Wire Wire Line
+	2600 2800 2800 2800
+Connection ~ 2800 2800
+Wire Wire Line
+	2800 3100 2800 3200
+Wire Wire Line
+	3100 2900 3100 3200
+Wire Wire Line
+	3100 3200 2800 3200
+Connection ~ 2800 3200
+Wire Wire Line
+	2800 3200 2800 3750
+Wire Wire Line
+	2050 3600 2600 3600
+Wire Wire Line
+	2050 3750 2800 3750
+Wire Wire Line
+	2200 2600 4400 2600
+Wire Wire Line
+	2800 2800 4400 2800
+Wire Wire Line
+	3100 2900 4400 2900
+$Comp
+L Device:R_Small R?
+U 1 1 5BB273AF
+P 3450 3300
+F 0 "R?" H 3509 3346 50  0000 L CNN
+F 1 "1K" H 3509 3255 50  0000 L CNN
+F 2 "" H 3450 3300 50  0001 C CNN
+F 3 "~" H 3450 3300 50  0001 C CNN
+	1    3450 3300
+	1    0    0    -1
+$EndComp
+Text HLabel 3350 3100 0    50   Input ~ 0
+Vcc
+Wire Wire Line
+	3350 3100 3450 3100
+Wire Wire Line
+	3450 3100 3450 3200
+Text HLabel 2000 4150 0    50   Input ~ 0
+R_Sense
+$Comp
+L Switch:SW_SPDT SW?
+U 1 1 5BB28D71
+P 3750 3700
+F 0 "SW?" V 3700 3500 50  0000 L CNN
+F 1 "SW_SPDT" V 3650 3800 50  0000 L CNN
+F 2 "" H 3750 3700 50  0001 C CNN
+F 3 "" H 3750 3700 50  0001 C CNN
+	1    3750 3700
+	0    1    1    0
+$EndComp
+Wire Wire Line
+	3450 3400 3450 4150
+Wire Wire Line
+	3750 3500 3750 3000
+Wire Wire Line
+	3750 3000 4400 3000
+Wire Wire Line
+	2000 4150 3450 4150
+Wire Wire Line
+	3650 3900 3650 4150
+Wire Wire Line
+	3650 4150 3450 4150
+Connection ~ 3450 4150
+Text HLabel 2000 4350 0    50   Input ~ 0
+T_Sense
+Wire Wire Line
+	2000 4350 3850 4350
+Wire Wire Line
+	3850 4350 3850 3900
+$Comp
+L Device:R_Small R_4_20
+U 1 1 5BB2D134
+P 4500 4350
+F 0 "R_4_20" V 4600 4350 50  0000 C CNN
+F 1 "100" V 4395 4350 50  0000 C CNN
+F 2 "" H 4500 4350 50  0001 C CNN
+F 3 "~" H 4500 4350 50  0001 C CNN
+	1    4500 4350
+	0    1    1    0
+$EndComp
+Text HLabel 2000 4600 0    50   Input ~ 0
+420+
+Text HLabel 2000 4800 0    50   Input ~ 0
+420-
+Wire Wire Line
+	4400 3200 4250 3200
+Wire Wire Line
+	4250 3200 4250 4350
+Wire Wire Line
+	4250 4600 2000 4600
+Wire Wire Line
+	4400 3300 4350 3300
+Wire Wire Line
+	4350 3300 4350 4050
+Wire Wire Line
+	4350 4050 4700 4050
+Wire Wire Line
+	4700 4050 4700 4350
+Wire Wire Line
+	4700 4800 2000 4800
+Wire Wire Line
+	4400 4350 4250 4350
+Connection ~ 4250 4350
+Wire Wire Line
+	4250 4350 4250 4600
+Wire Wire Line
+	4600 4350 4700 4350
+Connection ~ 4700 4350
+Wire Wire Line
+	4700 4350 4700 4800
 $EndSCHEMATC

Commit message: Changes: 1. RPi hierarchial sheet populated with appropriate circuit 2. Wiring hierarchial sheets together completed except for the temperature sensor
Connections:
- net labels removed: V_Sense
Changed lines of the file:
@@
 Title ""
 Date "2018-10-01"
-Rev "0.4"
+Rev "0.5"
 Comp "Bodhileaf Technologies"
 Comment1 ""
@@
 Text HLabel 2200 3250 3    50   BiDi ~ 0
 Gnd
-Text HLabel 2000 2250 0    50   Input ~ 0
-V_Sense
-Wire Wire Line
-	2000 2250 2200 2250
-Wire Wire Line
-	2200 2250 2200 2350
 Wire Wire Line
 	2200 2900 2200 2850
@@
 Wire Wire Line
 	4700 4350 4700 4800
+Wire Wire Line
+	2200 1750 4800 1750
+Wire Wire Line
+	2200 1750 2200 2350
 $EndSCHEMATC

Commit message: Changes: 1. Added all component footprints
Parts:
- removed C?: 0.1uF, 0.1uF, symbol Device:CP1_Small
- removed R?: 20m, symbol Device:R_Small
- removed SW?: SW_SPDT, symbol Switch:SW_SPDT
- added C2: 0.1uF, Capacitor_SMD:C_1206_3216Metric, symbol Device:C_Small
- added R20, R6: 0Ohms, Resistor_SMD:R_0805_2012Metric, symbol Device:R_Small
- C1: renamed from C?; footprint (none) -> Capacitor_Tantalum_SMD:CP_EIA-3216-12_Kemet-S
- R3, R4, R5: renamed from R?; footprint (none) -> Resistor_SMD:R_1206_3216Metric
- R7: renamed from R?; footprint (none) -> Resistor_SMD:R_0805_2012Metric
- R_4_20: footprint (none) -> Resistor_SMD:R_1206_3216Metric
- U5: renamed from U?; footprint (none) -> Package_SO:SOIC-14W_7.5x9.0mm_P1.27mm
Connections:
- wire segments 59 -> 60
Changed lines of the file:
@@
 $EndDescr
 $Comp
-L Analog_ADC:MCP3428 U?
+L Analog_ADC:MCP3428 U5
 U 1 1 5BB12D76
 P 4800 2900
-F 0 "U?" H 4550 3350 50  0000 C CNN
+F 0 "U5" H 4550 3350 50  0000 C CNN
 F 1 "MCP3428" H 5050 3350 50  0000 C CNN
-F 2 "" H 4800 2900 50  0001 C CNN
+F 2 "Package_SO:SOIC-14W_7.5x9.0mm_P1.27mm" H 4800 2900 50  0001 C CNN
 F 3 "http://ww1.microchip.com/downloads/en/DeviceDoc/22226a.pdf" H 4800 2900 50  0001 C CNN
 	1    4800 2900
@@
 $EndComp
 $Comp
-L Device:CP1_Small C?
-U 1 1 5BB12E03
-P 5500 1950
-F 0 "C?" H 5591 1996 50  0000 L CNN
-F 1 "0.1uF" H 5591 1905 50  0000 L CNN
-F 2 "0.1uF" H 5500 1950 50  0001 C CNN
-F 3 "~" H 5500 1950 50  0001 C CNN
-	1    5500 1950
-	1    0    0    -1
-$EndComp
-$Comp
-L Device:CP_Small C?
+L Device:CP_Small C1
 U 1 1 5BB12EC2
 P 5100 1950
-F 0 "C?" H 5188 1996 50  0000 L CNN
+F 0 "C1" H 5188 1996 50  0000 L CNN
 F 1 "10uF" H 5188 1905 50  0000 L CNN
-F 2 "" H 5100 1950 50  0001 C CNN
+F 2 "Capacitor_Tantalum_SMD:CP_EIA-3216-12_Kemet-S" H 5100 1950 50  0001 C CNN
 F 3 "~" H 5100 1950 50  0001 C CNN
 	1    5100 1950
@@
 Gnd
 $Comp
-L Device:R_Small R?
+L Device:R_Small R3
 U 1 1 5BB20FA7
 P 2200 2450
-F 0 "R?" H 2259 2496 50  0000 L CNN
+F 0 "R3" H 2259 2496 50  0000 L CNN
 F 1 "10K" H 2259 2405 50  0000 L CNN
-F 2 "" H 2200 2450 50  0001 C CNN
+F 2 "Resistor_SMD:R_1206_3216Metric" H 2200 2450 50  0001 C CNN
 F 3 "~" H 2200 2450 50  0001 C CNN
 	1    2200 2450
@@
 $EndComp
 $Comp
-L Device:R_Small R?
+L Device:R_Small R4
 U 1 1 5BB20FD7
 P 2200 2750
-F 0 "R?" H 2259 2796 50  0000 L CNN
+F 0 "R4" H 2259 2796 50  0000 L CNN
 F 1 "10K" H 2259 2705 50  0000 L CNN
-F 2 "" H 2200 2750 50  0001 C CNN
+F 2 "Resistor_SMD:R_1206_3216Metric" H 2200 2750 50  0001 C CNN
 F 3 "~" H 2200 2750 50  0001 C CNN
 	1    2200 2750
@@
 	2200 2600 2200 2550
 $Comp
-L Device:R_Small R?
+L Device:R_Small R5
 U 1 1 5BB21FC0
 P 2200 3000
-F 0 "R?" H 2259 3046 50  0000 L CNN
+F 0 "R5" H 2259 3046 50  0000 L CNN
 F 1 "10K" H 2259 2955 50  0000 L CNN
-F 2 "" H 2200 3000 50  0001 C CNN
+F 2 "Resistor_SMD:R_1206_3216Metric" H 2200 3000 50  0001 C CNN
 F 3 "~" H 2200 3000 50  0001 C CNN
 	1    2200 3000
@@
 Wire Wire Line
 	2200 3100 2200 3250
-$Comp
-L Device:R_Small R?
-U 1 1 5BB22A1E
-P 2800 3000
-F 0 "R?" H 2859 3046 50  0000 L CNN
-F 1 "20m" H 2859 2955 50  0000 L CNN
-F 2 "" H 2800 3000 50  0001 C CNN
-F 3 "~" H 2800 3000 50  0001 C CNN
-	1    2800 3000
-	1    0    0    -1
-$EndComp
-Wire Wire Line
-	2800 2900 2800 2800
 Text HLabel 2050 3600 0    50   Input ~ 0
 I_Sense+
@@
 	2600 3600 2600 2800
 Wire Wire Line
-	2600 2800 2800 2800
-Connection ~ 2800 2800
-Wire Wire Line
-	2800 3100 2800 3200
-Wire Wire Line
 	3100 2900 3100 3200
 Wire Wire Line
 	3100 3200 2800 3200
-Connection ~ 2800 3200
 Wire Wire Line
 	2800 3200 2800 3750
@@
 	2200 2600 4400 2600
 Wire Wire Line
-	2800 2800 4400 2800
-Wire Wire Line
 	3100 2900 4400 2900
 $Comp
-L Device:R_Small R?
+L Device:R_Small R7
 U 1 1 5BB273AF
 P 3450 3300
-F 0 "R?" H 3509 3346 50  0000 L CNN
+F 0 "R7" H 3509 3346 50  0000 L CNN
 F 1 "1K" H 3509 3255 50  0000 L CNN
-F 2 "" H 3450 3300 50  0001 C CNN
+F 2 "Resistor_SMD:R_0805_2012Metric" H 3450 3300 50  0001 C CNN
 F 3 "~" H 3450 3300 50  0001 C CNN
 	1    3450 3300
@@
 Text HLabel 2000 4150 0    50   Input ~ 0
 R_Sense
-$Comp
-L Switch:SW_SPDT SW?
-U 1 1 5BB28D71
-P 3750 3700
-F 0 "SW?" V 3700 3500 50  0000 L CNN
-F 1 "SW_SPDT" V 3650 3800 50  0000 L CNN
-F 2 "" H 3750 3700 50  0001 C CNN
-F 3 "" H 3750 3700 50  0001 C CNN
-	1    3750 3700
-	0    1    1    0
-$EndComp
 Wire Wire Line
 	3450 3400 3450 4150
@@
 Wire Wire Line
 	2000 4150 3450 4150
-Wire Wire Line
-	3650 3900 3650 4150
 Wire Wire Line
 	3650 4150 3450 4150
@@
 Wire Wire Line
 	2000 4350 3850 4350
-Wire Wire Line
-	3850 4350 3850 3900
 $Comp
 L Device:R_Small R_4_20
@@
 F 0 "R_4_20" V 4600 4350 50  0000 C CNN
 F 1 "100" V 4395 4350 50  0000 C CNN
-F 2 "" H 4500 4350 50  0001 C CNN
+F 2 "Resistor_SMD:R_1206_3216Metric" H 4500 4350 50  0001 C CNN
 F 3 "~" H 4500 4350 50  0001 C CNN
 	1    4500 4350
@@
 Wire Wire Line
 	2200 1750 2200 2350
+$Comp
+L Device:C_Small C2
+U 1 1 5BB4702F
+P 5500 1950
+F 0 "C2" H 5592 1996 50  0000 L CNN
+F 1 "0.1uF" H 5592 1905 50  0000 L CNN
+F 2 "Capacitor_SMD:C_1206_3216Metric" H 5500 1950 50  0001 C CNN
+F 3 "~" H 5500 1950 50  0001 C CNN
+	1    5500 1950
+	1    0    0    -1
+$EndComp
+Wire Wire Line
+	2600 2800 4400 2800
+$Comp
+L Device:R_Small R6
+U 1 1 5BB4E9C6
+P 3650 3700
+F 0 "R6" H 3500 3600 50  0000 L CNN
+F 1 "0Ohms" V 3550 3650 50  0000 L CNN
+F 2 "Resistor_SMD:R_0805_2012Metric" H 3650 3700 50  0001 C CNN
+F 3 "~" H 3650 3700 50  0001 C CNN
+	1    3650 3700
+	1    0    0    -1
+$EndComp
+$Comp
+L Device:R_Small R20
+U 1 1 5BB4EB74
+P 3850 3700
+F 0 "R20" H 3950 3600 50  0000 L CNN
+F 1 "0Ohms" V 3950 3650 50  0000 L CNN
+F 2 "Resistor_SMD:R_0805_2012Metric" H 3850 3700 50  0001 C CNN
+F 3 "~" H 3850 3700 50  0001 C CNN
+	1    3850 3700
+	1    0    0    -1
+$EndComp
+Wire Wire Line
+	3750 3500 3650 3500
+Wire Wire Line
+	3650 3500 3650 3600
+Wire Wire Line
+	3650 3800 3650 4150
+Wire Wire Line
+	3750 3500 3850 3500
+Wire Wire Line
+	3850 3500 3850 3600
+Connection ~ 3750 3500
+Wire Wire Line
+	3850 3800 3850 4350
 $EndSCHEMATC

Commit message: Changes: 1. Removed TVS diodes in favour of a RS485 transceiver of the same footprint that contains ESD protection 2. Tried different layouts.
Parts:
- C2: footprint Capacitor_SMD:C_1206_3216Metric -> Capacitor_SMD:C_0805_2012Metric
Changed lines of the file:
@@
 F 0 "C2" H 5592 1996 50  0000 L CNN
 F 1 "0.1uF" H 5592 1905 50  0000 L CNN
-F 2 "Capacitor_SMD:C_1206_3216Metric" H 5500 1950 50  0001 C CNN
+F 2 "Capacitor_SMD:C_0805_2012Metric" H 5500 1950 50  0001 C CNN
 F 3 "~" H 5500 1950 50  0001 C CNN
 	1    5500 1950

Commit message: Changes: 1. Laid out the ADC part 2. Removed an unnecessary 10K resistor in the ADC voltage sense part
Parts:
- removed R5: 10K, Resistor_SMD:R_1206_3216Metric, symbol Device:R_Small
Connections:
- wire segments 60 -> 59
Changed lines of the file:
@@
 	1    0    0    -1
 $EndComp
-Text HLabel 2200 3250 3    50   BiDi ~ 0
+Text HLabel 2200 3050 3    50   BiDi ~ 0
 Gnd
-Wire Wire Line
-	2200 2900 2200 2850
 Wire Wire Line
 	2200 2650 2200 2600
@@
 Wire Wire Line
 	2200 2600 2200 2550
-$Comp
-L Device:R_Small R5
-U 1 1 5BB21FC0
-P 2200 3000
-F 0 "R5" H 2259 3046 50  0000 L CNN
-F 1 "10K" H 2259 2955 50  0000 L CNN
-F 2 "Resistor_SMD:R_1206_3216Metric" H 2200 3000 50  0001 C CNN
-F 3 "~" H 2200 3000 50  0001 C CNN
-	1    2200 3000
-	1    0    0    -1
-$EndComp
-Wire Wire Line
-	2200 3100 2200 3250
 Text HLabel 2050 3600 0    50   Input ~ 0
 I_Sense+
@@
 Wire Wire Line
 	3850 3800 3850 4350
+Wire Wire Line
+	2200 2850 2200 3050
 $EndSCHEMATC
