File: analogSensing.sch (KiCad schematic (older format))
At the start: 9 parts, among them U5 MCP3428

Commit message: Changes: 1. Added a power LED 2. Added PPTC to the inputs of optocoupler 3. Added PPTC to the transceiver side of the RS232 driver 4. Corrected ADC footprint
Parts:
- U5: footprint Package_SO:SOIC-14W_7.5x9.0mm_P1.27mm -> Package_SO:SOIC-14_3.9x8.7mm_P1.27mm
Changed lines of the file:
@@
 F 0 "U5" H 4550 3350 50  0000 C CNN
 F 1 "MCP3428" H 5050 3350 50  0000 C CNN
-F 2 "Package_SO:SOIC-14W_7.5x9.0mm_P1.27mm" H 4800 2900 50  0001 C CNN
+F 2 "Package_SO:SOIC-14_3.9x8.7mm_P1.27mm" H 4800 2900 50  0001 C CNN
 F 3 "http://ww1.microchip.com/downloads/en/DeviceDoc/22226a.pdf" H 4800 2900 50  0001 C CNN
 	1    4800 2900
