File: powerSupply.sch (KiCad schematic (older format))
At the start: 11 parts

Commit message: Changes: 1. Serial (RS232, 485) circuit added.
Parts:
- added J?: Battery_Backup_Bypass, symbol Connector:Conn_01x02_Male
Connections:
- wire segments 45 -> 47
Changed lines of the file:
@@
 EESchema Schematic File Version 4
+LIBS:sanjaya-cache
 EELAYER 26 0
 EELAYER END
@@
 Sheet 2 7
 Title "Power Supply"
-Date "2018-09-25"
-Rev "0.1"
+Date "2018-09-29"
+Rev "0.2"
 Comp "Bodhileaf Technologies"
 Comment1 ""
@@
 Wire Wire Line
 	3450 1400 6500 1400
+$Comp
+L Connector:Conn_01x02_Male J?
+U 1 1 5BAE59DD
+P 7550 3800
+F 0 "J?" V 7703 3612 50  0000 R CNN
+F 1 "Battery_Backup_Bypass" V 7612 3612 50  0000 R CNN
+F 2 "" H 7550 3800 50  0001 C CNN
+F 3 "~" H 7550 3800 50  0001 C CNN
+	1    7550 3800
+	0    -1   -1   0
+$EndComp
+Wire Wire Line
+	7100 3600 7550 3600
+Connection ~ 7100 3600
+Wire Wire Line
+	7650 3600 8100 3600
+Connection ~ 8100 3600
 $EndSCHEMATC

Commit message: Changes: 1. Added all component footprints
Parts:
- removed J?: USB_A, symbol Connector:USB_A
- added J9: USB_B_Micro_IN, Connector_USB:USB_Micro-B_GCT_USB3076-30-A, symbol Connector:USB_B_Micro
- D1: renamed from D?; footprint (none) -> Diode_SMD:D_SOT-23_ANK
- D2: renamed from D?; footprint (none) -> Diode_SMD:D_SMA
- F1: renamed from F?; footprint (none) -> Fuse:Fuse_1210_3225Metric
- J10, J8: renamed from J?; footprint (none) -> Resistor_SMD:R_0805_2012Metric
- J11: renamed from J?; value USB_B_Micro -> USB_B_Micro_OUT; footprint (none) -> Connector_USB:USB_Micro-B_GCT_USB3076-30-A
- J12: renamed from J?; footprint (none) -> Connector_JST:JST_EH_B02B-EH-A_1x02_P2.50mm_Vertical
- Q1: renamed from Q?; footprint (none) -> Package_TO_SOT_SMD:SOT-23
- Q2: renamed from Q?; footprint (none) -> Package_TO_SOT_SMD:SuperSOT-6
- R2: renamed from R?; footprint (none) -> Resistor_SMD:R_0805_2012Metric
- U3: renamed from U?; footprint (none) -> Package_TO_SOT_SMD:SOT-23-5
Connections:
- no-connect marks 7 -> 8
Changed lines of the file:
@@
 V_adapter_out
 $Comp
-L Device:Q_PMOS_GSD Q?
+L Device:Q_PMOS_GSD Q1
 U 1 1 5BAA5E31
 P 2500 1900
-F 0 "Q?" V 2843 1900 50  0000 C CNN
+F 0 "Q1" V 2843 1900 50  0000 C CNN
 F 1 "Q_PMOS_GSD" V 2752 1900 50  0000 C CNN
-F 2 "" H 2700 2000 50  0001 C CNN
+F 2 "Package_TO_SOT_SMD:SOT-23" H 2700 2000 50  0001 C CNN
 F 3 "~" H 2500 1900 50  0001 C CNN
 	1    2500 1900
@@
 $EndComp
 $Comp
-L Device:D_Zener_Small D?
+L Device:D_Zener_Small D1
 U 1 1 5BAA62D5
 P 2950 2000
-F 0 "D?" V 2904 2068 50  0000 L CNN
+F 0 "D1" V 2904 2068 50  0000 L CNN
 F 1 "10V" V 2995 2068 50  0000 L CNN
-F 2 "" V 2950 2000 50  0001 C CNN
+F 2 "Diode_SMD:D_SOT-23_ANK" V 2950 2000 50  0001 C CNN
 F 3 "~" V 2950 2000 50  0001 C CNN
 	1    2950 2000
@@
 $EndComp
 $Comp
-L Device:Fuse F?
+L Device:Fuse F1
 U 1 1 5BAA63D1
 P 1950 1800
-F 0 "F?" V 1753 1800 50  0000 C CNN
+F 0 "F1" V 1753 1800 50  0000 C CNN
 F 1 "3A" V 1844 1800 50  0000 C CNN
-F 2 "" V 1880 1800 50  0001 C CNN
+F 2 "Fuse:Fuse_1210_3225Metric" V 1880 1800 50  0001 C CNN
 F 3 "~" H 1950 1800 50  0001 C CNN
 	1    1950 1800
@@
 $EndComp
 $Comp
-L Device:R_Small R?
+L Device:R_Small R2
 U 1 1 5BAA651A
 P 2500 2800
-F 0 "R?" H 2559 2846 50  0000 L CNN
+F 0 "R2" H 2559 2846 50  0000 L CNN
 F 1 "10K" H 2559 2755 50  0000 L CNN
-F 2 "" H 2500 2800 50  0001 C CNN
+F 2 "Resistor_SMD:R_0805_2012Metric" H 2500 2800 50  0001 C CNN
 F 3 "~" H 2500 2800 50  0001 C CNN
 	1    2500 2800
@@
 $EndComp
 $Comp
-L Device:D_Zener D?
+L Device:D_Zener D2
 U 1 1 5BAA66A0
 P 3400 2050
-F 0 "D?" V 3354 2129 50  0000 L CNN
+F 0 "D2" V 3354 2129 50  0000 L CNN
 F 1 "24V" V 3445 2129 50  0000 L CNN
-F 2 "" H 3400 2050 50  0001 C CNN
+F 2 "Diode_SMD:D_SMA" H 3400 2050 50  0001 C CNN
 F 3 "~" H 3400 2050 50  0001 C CNN
 	1    3400 2050
@@
 	2500 2100 2500 2250
 $Comp
-L Custom_Discrete:FDC021N30 Q?
+L Custom_Discrete:FDC021N30 Q2
 U 1 1 5BAB38D4
 P 5400 2150
-F 0 "Q?" V 5421 1822 50  0000 R CNN
+F 0 "Q2" V 5421 1822 50  0000 R CNN
 F 1 "FDC021N30" V 5330 1822 50  0000 R CNN
-F 2 "" H 5400 1850 50  0001 C CNN
+F 2 "Package_TO_SOT_SMD:SuperSOT-6" H 5400 1850 50  0001 C CNN
 F 3 "https://www.mouser.in/datasheet/2/308/FDC021N30-1119132.pdf" H 5400 1850 50  0001 C CNN
 	1    5400 2150
@@
 $EndComp
 $Comp
-L Custom_ICs:TPS2400BVR U?
+L Custom_ICs:TPS2400BVR U3
 U 1 1 5BAB3A2A
 P 4450 3150
-F 0 "U?" H 4878 3196 50  0000 L CNN
+F 0 "U3" H 4878 3196 50  0000 L CNN
 F 1 "TPS2400BVR" H 4878 3105 50  0000 L CNN
-F 2 "" H 4450 3150 50  0001 C CNN
+F 2 "Package_TO_SOT_SMD:SOT-23-5" H 4450 3150 50  0001 C CNN
 F 3 "" H 4450 3150 50  0001 C CNN
 	1    4450 3150
@@
 Connection ~ 6500 1800
 $Comp
-L Connector:USB_A J?
-U 1 1 5BAB59BB
-P 7100 2650
-F 0 "J?" H 7155 3117 50  0000 C CNN
-F 1 "USB_A" H 7155 3026 50  0000 C CNN
-F 2 "" H 7250 2600 50  0001 C CNN
-F 3 " ~" H 7250 2600 50  0001 C CNN
-	1    7100 2650
-	1    0    0    -1
-$EndComp
-$Comp
-L Connector:USB_B_Micro J?
+L Connector:USB_B_Micro J11
 U 1 1 5BAB5AB1
 P 8100 2650
-F 0 "J?" H 8155 3117 50  0000 C CNN
-F 1 "USB_B_Micro" H 8155 3026 50  0000 C CNN
-F 2 "" H 8250 2600 50  0001 C CNN
+F 0 "J11" H 8155 3117 50  0000 C CNN
+F 1 "USB_B_Micro_OUT" H 8155 3026 50  0000 C CNN
+F 2 "Connector_USB:USB_Micro-B_GCT_USB3076-30-A" H 8250 2600 50  0001 C CNN
 F 3 "~" H 8250 2600 50  0001 C CNN
 	1    8100 2650
@@
 NoConn ~ 8400 2850
 $Comp
-L Connector:Conn_01x02_Male J?
+L Connector:Conn_01x02_Male J12
 U 1 1 5BABDE81
 P 8900 2200
-F 0 "J?" H 8872 2080 50  0000 R CNN
+F 0 "J12" H 8872 2080 50  0000 R CNN
 F 1 "ON_Switch" H 8872 2171 50  0000 R CNN
-F 2 "" H 8900 2200 50  0001 C CNN
+F 2 "Connector_JST:JST_EH_B02B-EH-A_1x02_P2.50mm_Vertical" H 8900 2200 50  0001 C CNN
 F 3 "~" H 8900 2200 50  0001 C CNN
 	1    8900 2200
@@
 	8600 1800 9000 1800
 $Comp
-L Connector:Conn_01x02_Male J?
+L Connector:Conn_01x02_Male J8
 U 1 1 5BABF2C4
 P 3450 1000
-F 0 "J?" V 3510 1040 50  0000 L CNN
+F 0 "J8" V 3510 1040 50  0000 L CNN
 F 1 "Supply_Safety_Bypass" V 3601 1040 50  0000 L CNN
-F 2 "" H 3450 1000 50  0001 C CNN
+F 2 "Resistor_SMD:R_0805_2012Metric" H 3450 1000 50  0001 C CNN
 F 3 "~" H 3450 1000 50  0001 C CNN
 	1    3450 1000
@@
 	3450 1400 6500 1400
 $Comp
-L Connector:Conn_01x02_Male J?
+L Connector:Conn_01x02_Male J10
 U 1 1 5BAE59DD
 P 7550 3800
-F 0 "J?" V 7703 3612 50  0000 R CNN
+F 0 "J10" V 7703 3612 50  0000 R CNN
 F 1 "Battery_Backup_Bypass" V 7612 3612 50  0000 R CNN
-F 2 "" H 7550 3800 50  0001 C CNN
+F 2 "Resistor_SMD:R_0805_2012Metric" H 7550 3800 50  0001 C CNN
 F 3 "~" H 7550 3800 50  0001 C CNN
 	1    7550 3800
@@
 	7650 3600 8100 3600
 Connection ~ 8100 3600
+$Comp
+L Connector:USB_B_Micro J9
+U 1 1 5BB4D896
+P 7100 2650
+F 0 "J9" H 7155 3117 50  0000 C CNN
+F 1 "USB_B_Micro_IN" H 7155 3026 50  0000 C CNN
+F 2 "Connector_USB:USB_Micro-B_GCT_USB3076-30-A" H 7250 2600 50  0001 C CNN
+F 3 "~" H 7250 2600 50  0001 C CNN
+	1    7100 2650
+	1    0    0    -1
+$EndComp
+NoConn ~ 7400 2850
 $EndSCHEMATC

Commit message: Changes: 1. Some net names, connector names changed to be more meaningful 2. I2C connector added 3. Mistake in power bank bypass connection rectified 4. Layout changed. Almost finalized.
Parts:
- added J18: Bat_Bak_Byp_Vcc, Resistor_SMD:R_0805_2012Metric, symbol Connector:Conn_01x02_Male
- J10: value Battery_Backup_Bypass -> Bat_Bak_Byp_Gnd
Connections:
- wire segments 47 -> 51
Changed lines of the file:
@@
 Sheet 2 7
 Title "Power Supply"
-Date "2018-10-02"
-Rev "0.6"
+Date "2018-10-05"
+Rev "0.7"
 Comp "Bodhileaf Technologies"
 Comment1 ""
@@
 $EndComp
 Wire Wire Line
-	8400 2450 8600 2450
+	8400 2450 8550 2450
 Wire Wire Line
 	8600 2450 8600 2200
@@
 P 7550 3800
 F 0 "J10" V 7703 3612 50  0000 R CNN
-F 1 "Battery_Backup_Bypass" V 7612 3612 50  0000 R CNN
+F 1 "Bat_Bak_Byp_Gnd" V 7612 3612 50  0000 R CNN
 F 2 "Resistor_SMD:R_0805_2012Metric" H 7550 3800 50  0001 C CNN
 F 3 "~" H 7550 3800 50  0001 C CNN
@@
 $EndComp
 NoConn ~ 7400 2850
+$Comp
+L Connector:Conn_01x02_Male J18
+U 1 1 5BB845D3
+P 7800 1600
+F 0 "J18" V 7860 1640 50  0000 L CNN
+F 1 "Bat_Bak_Byp_Vcc" V 7951 1640 50  0000 L CNN
+F 2 "Resistor_SMD:R_0805_2012Metric" H 7800 1600 50  0001 C CNN
+F 3 "~" H 7800 1600 50  0001 C CNN
+	1    7800 1600
+	0    1    1    0
+$EndComp
+Wire Wire Line
+	7500 1800 7700 1800
+Connection ~ 7500 1800
+Wire Wire Line
+	7800 1800 8550 1800
+Wire Wire Line
+	8550 1800 8550 2450
+Connection ~ 8550 2450
+Wire Wire Line
+	8550 2450 8600 2450
 $EndSCHEMATC

Commit message: Changes: 1. Added a power LED 2. Added PPTC to the inputs of optocoupler 3. Added PPTC to the transceiver side of the RS232 driver 4. Corrected ADC footprint
Parts:
- D1: value 10V -> Zener_10V
- D2: value 24V -> Zener_24V
- F1: value 3A -> GlassFuse_3A; footprint Fuse:Fuse_1210_3225Metric -> Connector_JST:JST_EH_B02B-EH-A_1x02_P2.50mm_Vertical
Changed lines of the file:
@@
 P 2950 2000
 F 0 "D1" V 2904 2068 50  0000 L CNN
-F 1 "10V" V 2995 2068 50  0000 L CNN
+F 1 "Zener_10V" H 3000 2100 50  0000 L CNN
 F 2 "Diode_SMD:D_SOT-23_ANK" V 2950 2000 50  0001 C CNN
 F 3 "~" V 2950 2000 50  0001 C CNN
@@
 P 1950 1800
 F 0 "F1" V 1753 1800 50  0000 C CNN
-F 1 "3A" V 1844 1800 50  0000 C CNN
-F 2 "Fuse:Fuse_1210_3225Metric" V 1880 1800 50  0001 C CNN
+F 1 "GlassFuse_3A" V 1850 1750 50  0000 C CNN
+F 2 "Connector_JST:JST_EH_B02B-EH-A_1x02_P2.50mm_Vertical" V 1880 1800 50  0001 C CNN
 F 3 "~" H 1950 1800 50  0001 C CNN
 	1    1950 1800
@@
 P 3400 2050
 F 0 "D2" V 3354 2129 50  0000 L CNN
-F 1 "24V" V 3445 2129 50  0000 L CNN
+F 1 "Zener_24V" H 3450 2150 50  0000 L CNN
 F 2 "Diode_SMD:D_SMA" H 3400 2050 50  0001 C CNN
 F 3 "~" H 3400 2050 50  0001 C CNN
