File: digitalSensing.sch (KiCad schematic (older format))
At the start: 0 parts

Commit message: Changes: 1. Digital sensing circuit added.
Parts:
- added R? (x8): 1K, symbol Device:R_Small
- added U? (x4): TLP291-4, Package_DIP:SMDIP-16_W7.62mm, symbol Isolator:TLP291-4
- added U? (x5): 74HC14, symbol 74xx:74HC14
Connections:
- net labels added: Gnd_in, Gnd_out, Vcc, Vin_1, Vin_2, Vin_3, Vin_4, Vout_1, Vout_2, Vout_3, Vout_4
- wire segments 0 -> 47

Commit message: Changes: 1. Added all component footprints
Parts:
- R10, R11, R12, R13, R14, R15, R8, R9: renamed from R?; footprint (none) -> Resistor_SMD:R_0805_2012Metric
- U1: renamed from U?; footprint (none) -> Package_SO:TSSOP-14_4.4x5mm_P0.65mm
- U6: renamed from U?; footprint Package_DIP:SMDIP-16_W7.62mm -> Package_SO:SOP-16_4.4x10.4mm_P1.27mm
Changed lines of the file:
@@
 $EndDescr
 $Comp
-L Isolator:TLP291-4 U?
+L Isolator:TLP291-4 U6
 U 1 1 5BAF3DF5
 P 4200 3400
-F 0 "U?" H 4200 3725 50  0000 C CNN
+F 0 "U6" H 4200 3725 50  0000 C CNN
 F 1 "TLP291-4" H 4200 3634 50  0000 C CNN
-F 2 "Package_DIP:SMDIP-16_W7.62mm" H 4000 3200 50  0001 L CIN
+F 2 "Package_SO:SOP-16_4.4x10.4mm_P1.27mm" H 4000 3200 50  0001 L CIN
 F 3 "https://toshiba.semicon-storage.com/info/docget.jsp?did=12858&prodName=TLP291-4" H 4200 3400 50  0001 L CNN
 	1    4200 3400
@@
 $EndComp
 $Comp
-L Isolator:TLP291-4 U?
+L Isolator:TLP291-4 U6
 U 2 1 5BAF3E52
 P 4200 4000
-F 0 "U?" H 4200 4325 50  0000 C CNN
+F 0 "U6" H 4200 4325 50  0000 C CNN
 F 1 "TLP291-4" H 4200 4234 50  0000 C CNN
-F 2 "Package_DIP:SMDIP-16_W7.62mm" H 4000 3800 50  0001 L CIN
+F 2 "Package_SO:SOP-16_4.4x10.4mm_P1.27mm" H 4000 3800 50  0001 L CIN
 F 3 "https://toshiba.semicon-storage.com/info/docget.jsp?did=12858&prodName=TLP291-4" H 4200 4000 50  0001 L CNN
 	2    4200 4000
@@
 $EndComp
 $Comp
-L Isolator:TLP291-4 U?
+L Isolator:TLP291-4 U6
 U 3 1 5BAF3EE9
 P 4200 4600
-F 0 "U?" H 4200 4925 50  0000 C CNN
+F 0 "U6" H 4200 4925 50  0000 C CNN
 F 1 "TLP291-4" H 4200 4834 50  0000 C CNN
-F 2 "Package_DIP:SMDIP-16_W7.62mm" H 4000 4400 50  0001 L CIN
+F 2 "Package_SO:SOP-16_4.4x10.4mm_P1.27mm" H 4000 4400 50  0001 L CIN
 F 3 "https://toshiba.semicon-storage.com/info/docget.jsp?did=12858&prodName=TLP291-4" H 4200 4600 50  0001 L CNN
 	3    4200 4600
@@
 $EndComp
 $Comp
-L Isolator:TLP291-4 U?
+L Isolator:TLP291-4 U6
 U 4 1 5BAF3F76
 P 4200 5200
-F 0 "U?" H 4200 5525 50  0000 C CNN
+F 0 "U6" H 4200 5525 50  0000 C CNN
 F 1 "TLP291-4" H 4200 5434 50  0000 C CNN
-F 2 "Package_DIP:SMDIP-16_W7.62mm" H 4000 5000 50  0001 L CIN
+F 2 "Package_SO:SOP-16_4.4x10.4mm_P1.27mm" H 4000 5000 50  0001 L CIN
 F 3 "https://toshiba.semicon-storage.com/info/docget.jsp?did=12858&prodName=TLP291-4" H 4200 5200 50  0001 L CNN
 	4    4200 5200
@@
 $EndComp
 $Comp
-L Device:R_Small R?
+L Device:R_Small R8
 U 1 1 5BAF9096
 P 3700 3300
-F 0 "R?" V 3504 3300 50  0000 C CNN
+F 0 "R8" V 3504 3300 50  0000 C CNN
 F 1 "1K" V 3595 3300 50  0000 C CNN
-F 2 "" H 3700 3300 50  0001 C CNN
+F 2 "Resistor_SMD:R_0805_2012Metric" H 3700 3300 50  0001 C CNN
 F 3 "~" H 3700 3300 50  0001 C CNN
 	1    3700 3300
@@
 Gnd_in
 $Comp
-L Device:R_Small R?
+L Device:R_Small R9
 U 1 1 5BAFA5EA
 P 3700 3900
-F 0 "R?" V 3504 3900 50  0000 C CNN
+F 0 "R9" V 3504 3900 50  0000 C CNN
 F 1 "1K" V 3595 3900 50  0000 C CNN
-F 2 "" H 3700 3900 50  0001 C CNN
+F 2 "Resistor_SMD:R_0805_2012Metric" H 3700 3900 50  0001 C CNN
 F 3 "~" H 3700 3900 50  0001 C CNN
 	1    3700 3900
@@
 Gnd_in
 $Comp
-L Device:R_Small R?
+L Device:R_Small R10
 U 1 1 5BAFA63E
 P 3700 4500
-F 0 "R?" V 3504 4500 50  0000 C CNN
+F 0 "R10" V 3504 4500 50  0000 C CNN
 F 1 "1K" V 3595 4500 50  0000 C CNN
-F 2 "" H 3700 4500 50  0001 C CNN
+F 2 "Resistor_SMD:R_0805_2012Metric" H 3700 4500 50  0001 C CNN
 F 3 "~" H 3700 4500 50  0001 C CNN
 	1    3700 4500
@@
 Gnd_in
 $Comp
-L Device:R_Small R?
+L Device:R_Small R11
 U 1 1 5BAFA683
 P 3700 5100
-F 0 "R?" V 3504 5100 50  0000 C CNN
+F 0 "R11" V 3504 5100 50  0000 C CNN
 F 1 "1K" V 3595 5100 50  0000 C CNN
-F 2 "" H 3700 5100 50  0001 C CNN
+F 2 "Resistor_SMD:R_0805_2012Metric" H 3700 5100 50  0001 C CNN
 F 3 "~" H 3700 5100 50  0001 C CNN
 	1    3700 5100
@@
 	3800 5100 3900 5100
 $Comp
-L 74xx:74HC14 U?
+L 74xx:74HC14 U1
 U 1 1 5BAFD385
 P 5950 3300
-F 0 "U?" H 5950 3617 50  0000 C CNN
+F 0 "U1" H 5950 3617 50  0000 C CNN
 F 1 "74HC14" H 5950 3526 50  0000 C CNN
-F 2 "" H 5950 3300 50  0001 C CNN
+F 2 "Package_SO:TSSOP-14_4.4x5mm_P0.65mm" H 5950 3300 50  0001 C CNN
 F 3 "http://www.ti.com/lit/gpn/sn74HC14" H 5950 3300 50  0001 C CNN
 	1    5950 3300
@@
 $EndComp
 $Comp
-L 74xx:74HC14 U?
+L 74xx:74HC14 U1
 U 2 1 5BAFD3E9
 P 5950 3900
-F 0 "U?" H 5950 4217 50  0000 C CNN
+F 0 "U1" H 5950 4217 50  0000 C CNN
 F 1 "74HC14" H 5950 4126 50  0000 C CNN
-F 2 "" H 5950 3900 50  0001 C CNN
+F 2 "Package_SO:TSSOP-14_4.4x5mm_P0.65mm" H 5950 3900 50  0001 C CNN
 F 3 "http://www.ti.com/lit/gpn/sn74HC14" H 5950 3900 50  0001 C CNN
 	2    5950 3900
@@
 $EndComp
 $Comp
-L 74xx:74HC14 U?
+L 74xx:74HC14 U1
 U 3 1 5BAFD44A
 P 5950 4500
-F 0 "U?" H 5950 4817 50  0000 C CNN
+F 0 "U1" H 5950 4817 50  0000 C CNN
 F 1 "74HC14" H 5950 4726 50  0000 C CNN
-F 2 "" H 5950 4500 50  0001 C CNN
+F 2 "Package_SO:TSSOP-14_4.4x5mm_P0.65mm" H 5950 4500 50  0001 C CNN
 F 3 "http://www.ti.com/lit/gpn/sn74HC14" H 5950 4500 50  0001 C CNN
 	3    5950 4500
@@
 $EndComp
 $Comp
-L 74xx:74HC14 U?
+L 74xx:74HC14 U1
 U 4 1 5BAFD505
 P 5950 5100
-F 0 "U?" H 5950 5417 50  0000 C CNN
+F 0 "U1" H 5950 5417 50  0000 C CNN
 F 1 "74HC14" H 5950 5326 50  0000 C CNN
-F 2 "" H 5950 5100 50  0001 C CNN
+F 2 "Package_SO:TSSOP-14_4.4x5mm_P0.65mm" H 5950 5100 50  0001 C CNN
 F 3 "http://www.ti.com/lit/gpn/sn74HC14" H 5950 5100 50  0001 C CNN
 	4    5950 5100
@@
 $EndComp
 $Comp
-L 74xx:74HC14 U?
+L 74xx:74HC14 U1
 U 7 1 5BAFD574
 P 6350 1900
-F 0 "U?" H 6580 1946 50  0000 L CNN
+F 0 "U1" H 6580 1946 50  0000 L CNN
 F 1 "74HC14" H 6580 1855 50  0000 L CNN
-F 2 "" H 6350 1900 50  0001 C CNN
+F 2 "Package_SO:TSSOP-14_4.4x5mm_P0.65mm" H 6350 1900 50  0001 C CNN
 F 3 "http://www.ti.com/lit/gpn/sn74HC14" H 6350 1900 50  0001 C CNN
 	7    6350 1900
@@
 	6350 1300 6350 1400
 $Comp
-L Device:R_Small R?
+L Device:R_Small R12
 U 1 1 5BAFE49A
 P 5150 3150
-F 0 "R?" H 5091 3104 50  0000 R CNN
+F 0 "R12" H 5091 3104 50  0000 R CNN
 F 1 "1K" H 5091 3195 50  0000 R CNN
-F 2 "" H 5150 3150 50  0001 C CNN
+F 2 "Resistor_SMD:R_0805_2012Metric" H 5150 3150 50  0001 C CNN
 F 3 "~" H 5150 3150 50  0001 C CNN
 	1    5150 3150
@@
 $EndComp
 $Comp
-L Device:R_Small R?
+L Device:R_Small R13
 U 1 1 5BAFE4FF
 P 5150 3750
-F 0 "R?" H 5091 3704 50  0000 R CNN
+F 0 "R13" H 5091 3704 50  0000 R CNN
 F 1 "1K" H 5091 3795 50  0000 R CNN
-F 2 "" H 5150 3750 50  0001 C CNN
+F 2 "Resistor_SMD:R_0805_2012Metric" H 5150 3750 50  0001 C CNN
 F 3 "~" H 5150 3750 50  0001 C CNN
 	1    5150 3750
@@
 $EndComp
 $Comp
-L Device:R_Small R?
+L Device:R_Small R14
 U 1 1 5BAFE549
 P 5150 4350
-F 0 "R?" H 5091 4304 50  0000 R CNN
+F 0 "R14" H 5091 4304 50  0000 R CNN
 F 1 "1K" H 5091 4395 50  0000 R CNN
-F 2 "" H 5150 4350 50  0001 C CNN
+F 2 "Resistor_SMD:R_0805_2012Metric" H 5150 4350 50  0001 C CNN
 F 3 "~" H 5150 4350 50  0001 C CNN
 	1    5150 4350
@@
 $EndComp
 $Comp
-L Device:R_Small R?
+L Device:R_Small R15
 U 1 1 5BAFE591
 P 5150 4950
-F 0 "R?" H 5091 4904 50  0000 R CNN
+F 0 "R15" H 5091 4904 50  0000 R CNN
 F 1 "1K" H 5091 4995 50  0000 R CNN
-F 2 "" H 5150 4950 50  0001 C CNN
+F 2 "Resistor_SMD:R_0805_2012Metric" H 5150 4950 50  0001 C CNN
 F 3 "~" H 5150 4950 50  0001 C CNN
 	1    5150 4950

Commit message: Changes: 1. Added a power LED 2. Added PPTC to the inputs of optocoupler 3. Added PPTC to the transceiver side of the RS232 driver 4. Corrected ADC footprint
Parts:
- added F6, F7, F8, F9: PPTC_50mA, Fuse:Fuse_1210_3225Metric, symbol Device:Polyfuse_Small
Connections:
- wire segments 47 -> 51
Changed lines of the file:
@@
 	0    1    1    0
 $EndComp
-Text HLabel 3300 3300 0    50   Input ~ 0
+Text HLabel 2700 3300 0    50   Input ~ 0
 Vin_1
-Text HLabel 3300 3500 0    50   BiDi ~ 0
+Text HLabel 2700 3500 0    50   BiDi ~ 0
 Gnd_in
 $Comp
@@
 	0    1    1    0
 $EndComp
-Text HLabel 3300 3900 0    50   Input ~ 0
+Text HLabel 2700 3900 0    50   Input ~ 0
 Vin_2
-Text HLabel 3300 4100 0    50   BiDi ~ 0
+Text HLabel 2700 4100 0    50   BiDi ~ 0
 Gnd_in
 $Comp
@@
 	0    1    1    0
 $EndComp
-Text HLabel 3300 4500 0    50   Input ~ 0
+Text HLabel 2700 4500 0    50   Input ~ 0
 Vin_3
-Text HLabel 3300 4700 0    50   BiDi ~ 0
+Text HLabel 2700 4700 0    50   BiDi ~ 0
 Gnd_in
 $Comp
@@
 	0    1    1    0
 $EndComp
-Text HLabel 3300 5100 0    50   Input ~ 0
+Text HLabel 2700 5100 0    50   Input ~ 0
 Vin_4
-Text HLabel 3300 5300 0    50   BiDi ~ 0
+Text HLabel 2700 5300 0    50   BiDi ~ 0
 Gnd_in
 Wire Wire Line
-	3300 3300 3600 3300
-Wire Wire Line
 	3800 3300 3900 3300
 Wire Wire Line
-	3300 3500 3900 3500
-Wire Wire Line
 	3800 3900 3900 3900
 Wire Wire Line
-	3300 3900 3600 3900
-Wire Wire Line
-	3300 4100 3900 4100
-Wire Wire Line
-	3300 4500 3600 4500
-Wire Wire Line
-	3300 4700 3900 4700
-Wire Wire Line
 	3800 4500 3900 4500
-Wire Wire Line
-	3300 5100 3600 5100
-Wire Wire Line
-	3300 5300 3900 5300
 Wire Wire Line
 	3800 5100 3900 5100
@@
 Wire Wire Line
 	6250 5100 6450 5100
+$Comp
+L Device:Polyfuse_Small F6
+U 1 1 5BC05A3A
+P 3000 3300
+F 0 "F6" V 2795 3300 50  0000 C CNN
+F 1 "PPTC_50mA" V 2886 3300 50  0000 C CNN
+F 2 "Fuse:Fuse_1210_3225Metric" H 3050 3100 50  0001 L CNN
+F 3 "~" H 3000 3300 50  0001 C CNN
+	1    3000 3300
+	0    1    1    0
+$EndComp
+$Comp
+L Device:Polyfuse_Small F7
+U 1 1 5BC078FC
+P 3000 3900
+F 0 "F7" V 2795 3900 50  0000 C CNN
+F 1 "PPTC_50mA" V 2886 3900 50  0000 C CNN
+F 2 "Fuse:Fuse_1210_3225Metric" H 3050 3700 50  0001 L CNN
+F 3 "~" H 3000 3900 50  0001 C CNN
+	1    3000 3900
+	0    1    1    0
+$EndComp
+$Comp
+L Device:Polyfuse_Small F8
+U 1 1 5BC0794A
+P 3000 4500
+F 0 "F8" V 2795 4500 50  0000 C CNN
+F 1 "PPTC_50mA" V 2886 4500 50  0000 C CNN
+F 2 "Fuse:Fuse_1210_3225Metric" H 3050 4300 50  0001 L CNN
+F 3 "~" H 3000 4500 50  0001 C CNN
+	1    3000 4500
+	0    1    1    0
+$EndComp
+$Comp
+L Device:Polyfuse_Small F9
+U 1 1 5BC07996
+P 3000 5100
+F 0 "F9" V 2795 5100 50  0000 C CNN
+F 1 "PPTC_50mA" V 2886 5100 50  0000 C CNN
+F 2 "Fuse:Fuse_1210_3225Metric" H 3050 4900 50  0001 L CNN
+F 3 "~" H 3000 5100 50  0001 C CNN
+	1    3000 5100
+	0    1    1    0
+$EndComp
+Wire Wire Line
+	2700 3500 3900 3500
+Wire Wire Line
+	2700 3300 2900 3300
+Wire Wire Line
+	3100 3300 3600 3300
+Wire Wire Line
+	3100 3900 3600 3900
+Wire Wire Line
+	2700 3900 2900 3900
+Wire Wire Line
+	2700 4100 3900 4100
+Wire Wire Line
+	2700 4500 2900 4500
+Wire Wire Line
+	2700 4700 3900 4700
+Wire Wire Line
+	3100 4500 3600 4500
+Wire Wire Line
+	2700 5100 2900 5100
+Wire Wire Line
+	3100 5100 3600 5100
+Wire Wire Line
+	2700 5300 3900 5300
 $EndSCHEMATC
