File: digitalSensing.sch (KiCad schematic (older format))
At the start: 14 parts, among them U1 74HC14, U6 TLP291-4

Commit message: Changes: 1. Corrected RS485 circuit connections 2. Added silk screen labels and labels to schematics
Changed lines of the file:
@@
 Sheet 6 7
 Title ""
-Date "2018-10-17"
-Rev "0.9"
+Date "2018-11-24"
+Rev "0.91"
 Comp "Bodhileaf Technologies"
 Comment1 ""
@@
 	-1   0    0    1
 $EndComp
-Text HLabel 4400 2900 0    50   Input ~ 0
-Vcc
 Wire Wire Line
 	4900 2900 5150 2900
